File: hardware/MaTouch ESP32-S3 2.13“ Quad-Color Eink V1.1.brd (EAGLE design)
At the start: 59.2 x 29.2 mm, 111 parts, among them IC2 TP4054, J1 FPC24-80P-A, Q1 MOSFET-PCHANNEL, Q12 SI1308EDL, U3 ESP32-S3, U4 W25Q128JV, U5 SPX3819, X1 40MHz(10ppm)

Commit message: Update v1.1
Parts:
- moved J1 2.00 mm to (14.0, 14.6)
- moved C52 1.17 mm to (9.37, 7.98)
- moved S5 1.00 mm to (8.50, 26.2)
- moved C44 0.99 mm to (11.2, 11.4)
- moved C45 0.97 mm to (10.1, 11.4)
- moved C46 0.97 mm to (9.04, 11.3)
- moved C47 0.91 mm to (8.00, 11.3)
- moved R1 0.87 mm to (50.9, 23.5), turned to 270 degrees
- moved C49 0.61 mm to (8.00, 9.55), turned to 180 degrees
- moved ANT1 0.58 mm to (54.5, 21.5)
- moved C42 0.51 mm to (9.96, 6.71)
- moved D4 0.43 mm to (13.0, 10.5)
- moved C48 0.36 mm to (6.81, 11.3)
- moved R14 0.33 mm to (10.5, 5.69)
- moved C50 0.23 mm to (14.8, 9.55), turned to 0 degrees
Connections:
- net GND: no longer R1.1
- net IO1: now also R1.1
- net N$29: now also TF.P2
Routing:
- net N$71: track 6.49 -> 22.7 mm
- net IO1: track 0.00 -> 11.1 mm, vias 0 -> 2
- net +3V3: track 233.0 -> 239.5 mm
- net RESE: track 8.59 -> 11.9 mm
- net IO8: track 32.1 -> 34.2 mm
- net IO5: track 33.8 -> 35.8 mm
- net IO10: track 28.6 -> 30.6 mm
- net IO4: track 32.6 -> 34.6 mm
- net IO6: track 31.8 -> 33.8 mm
- net IO9: track 29.6 -> 31.6 mm
- net PREVGL: track 21.3 -> 19.8 mm
- net GDR: track 6.16 -> 4.85 mm
- net VCOM: track 18.4 -> 17.2 mm
- net N$10: track 15.9 -> 14.8 mm
- net N$22: track 11.0 -> 9.90 mm
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Other:
- board size 59.2 x 29.2 mm -> 60.4 x 29.2 mm
- board text added: "Quad-Color Eink V1.1"
- board text removed: "Quad-Color Eink V1.0"
