File: hardware/MaTouch ESP32-S3 2.13“ Quad-Color Eink V1.1.sch (EAGLE design)
At the start: 110 parts, among them IC2 TP4054, J1 FPC24-80P-A, Q1 MOSFET-PCHANNEL, Q12 SI1308EDL, U3 ESP32-S3, U4 W25Q128JV, U5 SPX3819, X1 40MHz(10ppm)

Commit message: Update v1.1
Connections:
- net GND: no longer R1.1
- net IO1: now also R1.1
- net N$29: now also TF.CD/DAT3
Other:
- note added: "ESP32-S3 EINK 2.13" v1.1"
- note removed: "ESP32-S3 EINK 2.13" v1.0"
- moved on the sheet: C16, C22, C26, C3, C31, C38, C39, C40, C41, C42, C43, C44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
